Commit message: Пункт 3 курсовой работы выполнен.
ADD: Добавлен файл README (Требование обеспечения вопроизводимых запусков)
UPD: Обновлена моделька башни на роботе.

ADD: Добавлен модуль fake_clock, чтобы синхронизировать симуляцию, и чтобы исправить ошибку с телепортированием робота и пропажей данных о положении.

File: src/my_robot_pkg/urdf/rviz_robot.urdf (robot description, URDF)
Before this commit: robot tank_robot, 8 links, 7 joints
Links:
- link tower_link: geometry collision box size=0.08 0.08 0.12; visual box size=0.08 0.08 0.12
Joints:
- joint laser_joint: origin xyz=0 0 0.12 rpy=0 0 0 -> xyz=0 0 0.145 rpy=0 0 0
